Commit message: edit nav2 bringup to load custom map and remove amcl

File: lr_ws/install/nav2_bringup/share/nav2_bringup/urdf/lr_rover.urdf (robot description, URDF)
Before this commit: robot 600220, 1 links, 0 joints
Links:
- link base_link: geometry visual mesh filename=file:///home/root/Lunar_ROADSTER/lr_ws/src/navigation2/nav2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 scale=0.001 0.001 0.001
